File: electronics/controlboard/controlboard.sch (KiCad schematic (older format))
At the start: 37 parts, among them J3 HLJ-6115ANL, P1 CONN_01X04, P2 FDI_Cable, P3 CONN_02X03, P4 CONN_02X03, P5 CONN_01X02, P7 CONN_02X02, U1 ONION-OMEGA2, U2 Recom_R78Cxx, U3 MAX98357A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

Commit message: KiCAD: correced library paths to reach the plan44-kicad library (when cloned from github into the same parent as pixelboard-hardware)
Parts:
- U1: symbol ONION-OMEGA2 -> ONION-OMEGA2-RESCUE-controlboard
Changed lines of the file:
@@
 LIBS:contrib
 LIBS:valves
-LIBS:ic-io
-LIBS:p44_pixelboard
-LIBS:plan44_from_eagle
+LIBS:plan44
 LIBS:controlboard-cache
 EELAYER 25 0
@@
 Date "2017-03-05"
 Rev "v4"
-Comp "plan44.ch"
+Comp "plan44.ch/luz"
 Comment1 ""
 Comment2 ""
@@
 $EndDescr
 $Comp
-L ONION-OMEGA2 U1
+L ONION-OMEGA2-RESCUE-controlboard U1
 U 1 1 57FDEEFD
 P 5800 2250
