File: electronics/touchboard/touchboard.sch (KiCad schematic (older format))
At the start: 27 parts, among them P1 CONN_02X03, P2 CONN_01X02, P3 CONN_01X02, U1 AT42QT1070, U2 MCP23017

Commit message: KiCAD: correced library paths to reach the plan44-kicad library (when cloned from github into the same parent as pixelboard-hardware)
Parts:
- U2: symbol MCP23S17 -> MCP23S17-RESCUE-touchboard
Changed lines of the file:
@@
 EESchema Schematic File Version 2
+LIBS:touchboard-rescue
 LIBS:power
 LIBS:device
@@
 LIBS:contrib
 LIBS:valves
-LIBS:ic-io
-LIBS:p44_pixelboard
-LIBS:plan44_from_eagle
+LIBS:plan44
 LIBS:touchboard-cache
 EELAYER 25 0
@@
 encoding utf-8
 Sheet 1 1
-Title ""
+Title "touchboard"
 Date ""
-Rev ""
-Comp ""
+Rev "v1"
+Comp "plan44.ch/luz"
 Comment1 ""
 Comment2 ""
@@
 $EndComp
 $Comp
-L MCP23S17 U2
+L MCP23S17-RESCUE-touchboard U2
 U 1 1 57FE8AAA
 P 7800 2700
